File: 03_voltage_channels.kicad_sch (KiCad schematic)
At the start: 16 parts, among them J1 1190370 16POS, J2 1190370 16POS, J3 1190370 16POS, K1 UD2-5NE, K10 UD2-5NE, K11 UD2-5NE, K12 UD2-5NE, K17 UD2-5NE, K2 UD2-5NE, K3 UD2-5NE, K4 UD2-5NE, K5 UD2-5NE, K6 UD2-5NE, K7 UD2-5NE, K8 UD2-5NE, K9 UD2-5NE

Commit message: Add Phoenix 1190370 connector footprint
Parts:
- J1, J2, J3: value 1190370 16POS -> Phoenix 1190370 8POS; footprint (none) -> BenchScan_Connectors:Phoenix_1190370_LPTA-2.5-8-5.0; symbol BenchScan_DMMX16-rescue:CONN16 -> BenchScan_DMMX16-rescue:CONN8
Connections:
- net CH10_HI: now also J3.3; no longer J3.5, J3.6
- net CH10_LO: now also J3.4; no longer J3.7, J3.8
- net CH11_HI: now also J3.5; no longer J3.10, J3.9
- net CH11_LO: now also J3.6; no longer J3.11, J3.12
- net CH12_HI: now also J3.7; no longer J3.13, J3.14
- net CH12_LO: now also J3.8; no longer J3.15, J3.16
- net CH1_HI: no longer J1.2
- net CH1_LO: now also J1.2; no longer J1.3, J1.4
- net CH2_HI: now also J1.3; no longer J1.5, J1.6
- net CH2_LO: now also J1.4; no longer J1.7, J1.8
- net CH3_HI: now also J1.5; no longer J1.10, J1.9
- net CH3_LO: now also J1.6; no longer J1.11, J1.12
- net CH4_HI: now also J1.7; no longer J1.13, J1.14
- net CH4_LO: now also J1.8; no longer J1.15, J1.16
- net CH5_HI: no longer J2.2
- net CH5_LO: now also J2.2; no longer J2.3, J2.4
- net CH6_HI: now also J2.3; no longer J2.5, J2.6
- net CH6_LO: now also J2.4; no longer J2.7, J2.8
- net CH7_HI: now also J2.5; no longer J2.10, J2.9
- net CH7_LO: now also J2.6; no longer J2.11, J2.12
- net CH8_HI: now also J2.7; no longer J2.13, J2.14
- net CH8_LO: now also J2.8; no longer J2.15, J2.16
- net CH9_HI: no longer J3.2
- net CH9_LO: now also J3.2; no longer J3.3, J3.4

Commit message: Assign custom footprints to schematic components
Parts:
- K1, K10, K11, K12, K17, K2, K3, K4, K5, K6, K7, K8, K9: footprint (none) -> BenchScan_Custom:Relay_KEMET_UD2_NE
Changed lines of the file:
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@@
 			)
 		)
-		(property "Footprint" ""
+		(property "Footprint" "BenchScan_Custom:Relay_KEMET_UD2_NE"
 			(at 39.37 132.08 0)
 			(hide yes)
@@
 			)
 		)
-		(property "Datasheet" ""
+		(property "Datasheet" "https://content.kemet.com/datasheets/KEM_R7005_UC2_UD2.pdf"
 			(at 39.37 132.08 0)
 			(hide yes)
@@
 			)
 		)
-		(property "Description" ""
+		(property "Description" "KEMET/YAGEO UD2-5NE low-power non-latching DPDT SMD signal relay"
 			(at 39.37 132.08 0)
 			(show_name no)
@@
 			)
 		)
-		(property "Footprint" ""
+		(property "Footprint" "BenchScan_Custom:Relay_KEMET_UD2_NE"
 			(at 95.25 132.08 0)
 			(hide yes)
@@
 			)
 		)
-		(property "Datasheet" ""
+		(property "Datasheet" "https://content.kemet.com/datasheets/KEM_R7005_UC2_UD2.pdf"
 			(at 95.25 132.08 0)
 			(hide yes)
@@
 			)
 		)
-		(property "Description" ""
+		(property "Description" "KEMET/YAGEO UD2-5NE low-power non-latching DPDT SMD signal relay"
 			(at 95.25 132.08 0)
 			(show_name no)
@@
 			)
 		)
-		(property "Footprint" ""
+		(property "Footprint" "BenchScan_Custom:Relay_KEMET_UD2_NE"
 			(at 151.13 132.08 0)
 			(hide yes)
@@
 			)
 		)
-		(property "Datasheet" ""
+		(property "Datasheet" "https://content.kemet.com/datasheets/KEM_R7005_UC2_UD2.pdf"
 			(at 151.13 132.08 0)
 			(hide yes)
@@
 			)
 		)
-		(property "Description" ""
+		(property "Description" "KEMET/YAGEO UD2-5NE low-power non-latching DPDT SMD signal relay"
 			(at 151.13 132.08 0)
 			(show_name no)
@@
 			)
 		)
-		(property "Footprint" ""
+		(property "Footprint" "BenchScan_Custom:Relay_KEMET_UD2_NE"
 			(at 207.01 132.08 0)
 			(hide yes)
@@
 			)
 		)
-		(property "Datasheet" ""
+		(property "Datasheet" "https://content.kemet.com/datasheets/KEM_R7005_UC2_UD2.pdf"
 			(at 207.01 132.08 0)
 			(hide yes)
@@
 			)
 		)
-		(property "Description" ""
+		(property "Description" "KEMET/YAGEO UD2-5NE low-power non-latching DPDT SMD signal relay"
 			(at 207.01 132.08 0)
 			(show_name no)
@@
 			)
 		)
-		(property "Footprint" ""
+		(property "Footprint" "BenchScan_Custom:Relay_KEMET_UD2_NE"
 			(at 262.89 132.08 0)
 			(hide yes)
@@
 			)
 		)
-		(property "Datasheet" ""
+		(property "Datasheet" "https://content.kemet.com/datasheets/KEM_R7005_UC2_UD2.pdf"
 			(at 262.89 132.08 0)
 			(hide yes)
@@
 			)
 		)
-		(property "Description" ""
+		(property "Description" "KEMET/YAGEO UD2-5NE low-power non-latching DPDT SMD signal relay"
 			(at 262.89 132.08 0)
 			(show_name no)
@@
 			)
 		)
-		(property "Footprint" ""
+		(property "Footprint" "BenchScan_Custom:Relay_KEMET_UD2_NE"
 			(at 318.77 132.08 0)
 			(hide yes)
@@
 			)
 		)
-		(property "Datasheet" ""
+		(property "Datasheet" "https://content.kemet.com/datasheets/KEM_R7005_UC2_UD2.pdf"
 			(at 318.77 132.08 0)
 			(hide yes)
@@
 			)
 		)
-		(property "Description" ""
+		(property "Description" "KEMET/YAGEO UD2-5NE low-power non-latching DPDT SMD signal relay"
 			(at 318.77 132.08 0)
 			(show_name no)
@@
 			)
 		)
-		(property "Footprint" ""
+		(property "Footprint" "BenchScan_Custom:Relay_KEMET_UD2_NE"
 			(at 40.64 186.69 0)
 			(hide yes)
@@
 			)
 		)
-		(property "Datasheet" ""
+		(property "Datasheet" "https://content.kemet.com/datasheets/KEM_R7005_UC2_UD2.pdf"
 			(at 40.64 186.69 0)
 			(hide yes)
@@
 			)
 		)
-		(property "Description" ""
+		(property "Description" "KEMET/YAGEO UD2-5NE low-power non-latching DPDT SMD signal relay"
 			(at 40.64 186.69 0)
 			(show_name no)
@@
 			)
 		)
-		(property "Footprint" ""
+		(property "Footprint" "BenchScan_Custom:Relay_KEMET_UD2_NE"
 			(at 96.52 186.69 0)
 			(hide yes)
@@
 			)
 		)
-		(property "Datasheet" ""
+		(property "Datasheet" "https://content.kemet.com/datasheets/KEM_R7005_UC2_UD2.pdf"
 			(at 96.52 186.69 0)
 			(hide yes)
@@
 			)
 		)
-		(property "Description" ""
+		(property "Description" "KEMET/YAGEO UD2-5NE low-power non-latching DPDT SMD signal relay"
 			(at 96.52 186.69 0)
 			(show_name no)
@@
 			)
 		)
-		(property "Footprint" ""
+		(property "Footprint" "BenchScan_Custom:Relay_KEMET_UD2_NE"
 			(at 152.4 186.69 0)
 			(hide yes)
@@
 			)
 		)
-		(property "Datasheet" ""
+		(property "Datasheet" "https://content.kemet.com/datasheets/KEM_R7005_UC2_UD2.pdf"
 			(at 152.4 186.69 0)
 			(hide yes)
@@
 			)
 		)
-		(property "Description" ""
+		(property "Description" "KEMET/YAGEO UD2-5NE low-power non-latching DPDT SMD signal relay"
 			(at 152.4 186.69 0)
 			(show_name no)
@@
 			)
 		)
-		(property "Footprint" ""
+		(property "Footprint" "BenchScan_Custom:Relay_KEMET_UD2_NE"
 			(at 208.28 186.69 0)
 			(hide yes)
@@
 			)
 		)
-		(property "Datasheet" ""
+		(property "Datasheet" "https://content.kemet.com/datasheets/KEM_R7005_UC2_UD2.pdf"
 			(at 208.28 186.69 0)
 			(hide yes)
@@
 			)
 		)
-		(property "Description" ""
+		(property "Description" "KEMET/YAGEO UD2-5NE low-power non-latching DPDT SMD signal relay"
 			(at 208.28 186.69 0)
 			(show_name no)
@@
 			)
 		)
-		(property "Footprint" ""
+		(property "Footprint" "BenchScan_Custom:Relay_KEMET_UD2_NE"
 			(at 264.16 186.69 0)
 			(hide yes)
@@
 			)
 		)
-		(property "Datasheet" ""
+		(property "Datasheet" "https://content.kemet.com/datasheets/KEM_R7005_UC2_UD2.pdf"
 			(at 264.16 186.69 0)
 			(hide yes)
@@
 			)
 		)
-		(property "Description" ""
+		(property "Description" "KEMET/YAGEO UD2-5NE low-power non-latching DPDT SMD signal relay"
 			(at 264.16 186.69 0)
 			(show_name no)
@@
 			)
 		)
-		(property "Footprint" ""
+		(property "Footprint" "BenchScan_Custom:Relay_KEMET_UD2_NE"
 			(at 320.04 186.69 0)
 			(hide yes)
@@
 			)
 		)
-		(property "Datasheet" ""
+		(property "Datasheet" "https://content.kemet.com/datasheets/KEM_R7005_UC2_UD2.pdf"
 			(at 320.04 186.69 0)
 			(hide yes)
@@
 			)
 		)
-		(property "Description" ""
+		(property "Description" "KEMET/YAGEO UD2-5NE low-power non-latching DPDT SMD signal relay"
 			(at 320.04 186.69 0)
 			(show_name no)
@@
 			)
 		)
-		(property "Footprint" ""
+		(property "Footprint" "BenchScan_Custom:Relay_KEMET_UD2_NE"
 			(at 374.65 186.69 0)
 			(hide yes)
@@
 			)
 		)
-		(property "Datasheet" ""
+		(property "Datasheet" "https://content.kemet.com/datasheets/KEM_R7005_UC2_UD2.pdf"
 			(at 374.65 186.69 0)
 			(hide yes)
@@
 			)
 		)
-		(property "Description" ""
+		(property "Description" "KEMET/YAGEO UD2-5NE low-power non-latching DPDT SMD signal relay"
 			(at 374.65 186.69 0)
 			(show_name no)
