File: 03_voltage_channels.kicad_sch (KiCad schematic)
At the start: 16 parts, among them J1 Phoenix 1190370 8POS, J2 Phoenix 1190370 8POS, J3 Phoenix 1190370 8POS, K1 UD2-5NE, K10 UD2-5NE, K11 UD2-5NE, K12 UD2-5NE, K17 UD2-5NE, K2 UD2-5NE, K3 UD2-5NE, K4 UD2-5NE, K5 UD2-5NE, K6 UD2-5NE, K7 UD2-5NE, K8 UD2-5NE, K9 UD2-5NE

Commit message: Correct J1-J4 Phoenix terminal footprints
Parts:
- J1, J2, J3: footprint BenchScan_Connectors:Phoenix_1190370_LPTA-2.5-8-5.0 -> BenchScan_Connectors:Phoenix_1190370_LPTA-2.5-8-5.0_16THT_Paired
Changed lines of the file:
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@@
 			)
 		)
-		(property "Footprint" "BenchScan_Connectors:Phoenix_1190370_LPTA-2.5-8-5.0"
+		(property "Footprint" "BenchScan_Connectors:Phoenix_1190370_LPTA-2.5-8-5.0_16THT_Paired"
 			(at 38.1 53.34 0)
 			(hide yes)
@@
 			)
 		)
-		(property "Footprint" "BenchScan_Connectors:Phoenix_1190370_LPTA-2.5-8-5.0"
+		(property "Footprint" "BenchScan_Connectors:Phoenix_1190370_LPTA-2.5-8-5.0_16THT_Paired"
 			(at 124.46 53.34 0)
 			(hide yes)
@@
 			)
 		)
-		(property "Footprint" "BenchScan_Connectors:Phoenix_1190370_LPTA-2.5-8-5.0"
+		(property "Footprint" "BenchScan_Connectors:Phoenix_1190370_LPTA-2.5-8-5.0_16THT_Paired"
 			(at 213.36 53.34 0)
 			(hide yes)
