File: 04_current_dmm_interface.kicad_sch (KiCad schematic)
At the start: 17 parts, among them J10 POMONA 73099 BLACK, J11 POMONA 73099 RED, J12 POMONA 73099 BLACK, J4 Phoenix 1190370 8POS, J5 691137710006 DMM, J6 POMONA 73099 RED, J8 POMONA 73099 BLACK, J9 POMONA 73099 RED, K13 UD2-5NE, K14 UD2-5NE, K15 UD2-5NE, K16 UD2-5NE

Commit message: Correct J1-J4 Phoenix terminal footprints
Parts:
- J4: footprint BenchScan_Connectors:Phoenix_1190370_LPTA-2.5-8-5.0 -> BenchScan_Connectors:Phoenix_1190370_LPTA-2.5-8-5.0_16THT_Paired
Changed lines of the file:
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@@
 			)
 		)
-		(property "Footprint" "BenchScan_Connectors:Phoenix_1190370_LPTA-2.5-8-5.0"
+		(property "Footprint" "BenchScan_Connectors:Phoenix_1190370_LPTA-2.5-8-5.0_16THT_Paired"
 			(at 99.06 64.77 0)
 			(hide yes)
